Commit message: added nav goals and pick/place goals. also added kitchen chair

File: urdf/coffee_table.urdf.xacro (robot description, xacro)
@@ -2,6 +2,7 @@
 <root xmlns:xacro="http://ros.org/wiki/xacro">
   <xacro:macro name="coffee_table" params="parent *origin">
+    <!-- Coffee table -->
     <joint name="${parent}_coffee_table_joint" type="fixed">
-      <xacro:insert_block name="origin" />
+      <origin xyz="3.345 2.99 0" rpy="0 0 ${M_PI/2}" />
       <parent link="${parent}" />
       <child link="coffee_table_link" />
@@ -9,5 +10,4 @@
     <link name="coffee_table_link">
       <visual>
-        <origin xyz="0.527 -2.546 0" rpy="0 0 ${M_PI/2}" />
         <geometry>
           <mesh filename="package://rail_collada_models/meshes/coffee_table.dae" />
@@ -15,4 +15,23 @@
       </visual>
     </link>
+    <joint name="${parent}_coffee_table_surface_joint" type="fixed">
+      <origin xyz="0 0 0.405" rpy="0 0 0"/>
+      <parent link="coffee_table_link"/>
+      <child link="coffee_table_surface_link"/>
+    </joint>
+      <link name="coffee_table_surface_link">
+      <visual>
+        <geometry>
+          <box size="0.1 0.1 0.1"/>
+        </geometry>
+      </visual>
+    </link>
+    <!-- coffee table nav goal, placed half of carl's length in front of the long side near the coffee_table2-->
+    <joint name="${parent}_coffee_table_nav_goal" type="fixed">
+      <origin xyz="0 0.6 0" rpy="0 0 0"/>
+      <parent link="coffee_table_link"/>
+      <child link="coffee_table_nav_goal_link"/>
+    </joint>
+    <xacro:nav_goal prefix="coffee_table"/>
   </xacro:macro>
 </root>

File: urdf/couch.urdf.xacro (robot description, xacro)
@@ -9,5 +9,5 @@
     <link name="couch_link">
       <visual>
-        <origin xyz="1.755 -2.68 0" rpy="0 0 ${M_PI/2}" />
+        <origin xyz="4.497 2.94 0" rpy="0 0 ${M_PI/2}" />
         <geometry>
           <mesh filename="package://rail_collada_models/meshes/couch.dae" />

File: urdf/ilab.urdf.xacro (robot description, xacro)
@@ -2,13 +2,14 @@
 <robot xmlns:xacro="http://www.ros.org/wiki/xacro" name="ilab">
   <xacro:include filename="$(find rail_collada_models)/urdf/kitchen_counter.urdf.xacro" />
+  <xacro:include filename="$(find rail_collada_models)/urdf/kitchen_chair.urdf.xacro" />
   <xacro:include filename="$(find rail_collada_models)/urdf/kitchen_table.urdf.xacro" />
   <xacro:include filename="$(find rail_collada_models)/urdf/coffee_table.urdf.xacro" />
-   <xacro:include filename="$(find rail_collada_models)/urdf/couch.urdf.xacro" />
-   <xacro:include filename="$(find rail_collada_models)/urdf/right_shelves.urdf.xacro" />
-   <xacro:include filename="$(find rail_collada_models)/urdf/tv.urdf.xacro" />
-   <xacro:include filename="$(find rail_collada_models)/urdf/left_shelves.urdf.xacro" />
-   <xacro:include filename="$(find rail_collada_models)/urdf/lazy_chair_1.urdf.xacro" />
-   <xacro:include filename="$(find rail_collada_models)/urdf/lazy_chair_2.urdf.xacro" />
-   <xacro:include filename="$(find rail_collada_models)/urdf/lab.urdf.xacro" />
+  <xacro:include filename="$(find rail_collada_models)/urdf/couch.urdf.xacro" />
+  <xacro:include filename="$(find rail_collada_models)/urdf/nav_goal.urdf.xacro" />
+  <xacro:include filename="$(find rail_collada_models)/urdf/right_shelves.urdf.xacro" />
+  <xacro:include filename="$(find rail_collada_models)/urdf/tv.urdf.xacro" />
+  <xacro:include filename="$(find rail_collada_models)/urdf/left_shelves.urdf.xacro" />
+  <xacro:include filename="$(find rail_collada_models)/urdf/lazy_chairs.urdf.xacro" />
+  <xacro:include filename="$(find rail_collada_models)/urdf/lab.urdf.xacro" />
   <xacro:property name="PARENT" value="map" />
   <xacro:property name="FRAME" value="ilab" />
@@ -26,29 +27,29 @@
   </xacro:lab>
   <xacro:kitchen_counter parent="${FRAME}">
-    <origin xyz="2.85 5.55 0" rpy="0 0 0" />
+    <origin xyz="0 0 0" rpy="0 0 0" />
   </xacro:kitchen_counter>
   <xacro:kitchen_table parent="${FRAME}">
-    <origin xyz="2.85 5.55 0" rpy="0 0 0" />
+    <origin xyz="0 0 0" rpy="0 0 0" />
   </xacro:kitchen_table>
   <xacro:coffee_table parent="${FRAME}">
-    <origin xyz="2.85 5.55 0" rpy="0 0 0" />
+    <origin xyz="0 0 0" rpy="0 0 0" />
   </xacro:coffee_table>
   <xacro:couch parent="${FRAME}">
-    <origin xyz="2.85 5.55 0" rpy="0 0 0" />
+    <origin xyz="0 0 0" rpy="0 0 0" />
   </xacro:couch>
   <xacro:right_shelves parent="${FRAME}">
-    <origin xyz="2.85 5.55 0" rpy="0 0 0" />
+    <origin xyz="0 0 0" rpy="0 0 0" />
   </xacro:right_shelves>
   <xacro:tv parent="${FRAME}">
-    <origin xyz="2.85 5.55 0" rpy="0 0 0" />
+    <origin xyz="0 0 0" rpy="0 0 0" />
   </xacro:tv>
   <xacro:left_shelves parent="${FRAME}">
-    <origin xyz="2.85 5.55 0" rpy="0 0 0" />
+    <origin xyz="0 0 0" rpy="0 0 0" />
   </xacro:left_shelves>
-  <xacro:lazy_chair_1 parent="${FRAME}">
-    <origin xyz="2.85 5.55 0" rpy="0 0 0" />
-  </xacro:lazy_chair_1>
-  <xacro:lazy_chair_2 parent="${FRAME}">
-    <origin xyz="2.85 5.55 0" rpy="0 0 0" />
-  </xacro:lazy_chair_2>
+  <xacro:lazy_chairs parent="${FRAME}">
+    <origin xyz="0 0 0" rpy="0 0 0" />
+  </xacro:lazy_chairs>
+  <xacro:kitchen_chair parent="${FRAME}">
+    <origin xyz="0 0 0" rpy="0 0 0" />
+  </xacro:kitchen_chair>
 </robot>

File: urdf/kitchen_counter.urdf.xacro (robot description, xacro)
@@ -2,17 +2,75 @@
 <root xmlns:xacro="http://ros.org/wiki/xacro">
   <xacro:macro name="kitchen_counter" params="parent *origin">
+    <!--Kitchen Counter -->
     <joint name="${parent}_kitchen_counter_joint" type="fixed">
-      <xacro:insert_block name="origin" />
+      <origin xyz="1.679 5.873 0" rpy="0 0 ${M_PI}"/>
       <parent link="${parent}" />
-      <child link="kitchen_counter_link" />
+      <child link="kitchen_counter_link"/>
     </joint>
     <link name="kitchen_counter_link">
       <visual>
-        <origin xyz="-1.229 .323 0" rpy="0 0 0" />
-        <geometry>
+         <geometry>
           <mesh filename="package://rail_collada_models/meshes/kitchen_counter.dae" />
         </geometry>
       </visual>
     </link>
+    <!-- Sink-->
+    <joint name="${parent}_sink_joint" type="fixed">
+      <origin xyz="0 0 0.92" rpy="0 0 0"/>
+      <parent link="kitchen_counter_link" />
+      <child link="sink_link"/>
+    </joint>
+    <link name="sink_link">
+      <visual>
+        <geometry>
+          <box size="0.1 0.1 0.1"/>
+        </geometry>
+      </visual>
+    </link>
+    <!-- Sink Nav Goal placed half of Carl's length in front of the middle of the sink-->
+    <joint name="${parent}_sink_nav_goal_joint" type="fixed">
+      <origin xyz="0 0.55 0" rpy="0 0 0"/>
+      <parent link="kitchen_counter_link" />
+      <child link="sink_nav_goal_link"/>
+    </joint>
+    <xacro:nav_goal prefix="sink"/>
+    <!-- LEFT -->
+    <joint name="${parent}_kitchen_counter_left_surface_joint" type="fixed">
+      <origin xyz="-0.6 0 0.92" rpy="0 0 0"/>
+      <parent link="kitchen_counter_link" />
+      <child link="kitchen_counter_left_surface_link"/>
+    </joint>
+    <link name="kitchen_counter_left_surface_link">
+      <visual>
+        <geometry>
+          <box size="0.1 0.1 0.1"/>
+        </geometry>
+      </visual>
+    </link>
+    <joint name= "${parent}_kitchen_counter_left_nav_goal_joint" type="fixed">
+      <origin xyz="-.6 0.55 0" rpy="0 0 0"/>
+      <parent link="kitchen_counter_link" />
+      <child link="kitchen_counter_left_nav_goal_link"/>
+    </joint>
+    <xacro:nav_goal prefix="kitchen_counter_left"/>
+    <!-- RIGHT -->
+    <joint name="${parent}_kitchen_counter_right_surface_joint" type="fixed">
+      <origin xyz="0.6 0 0.92" rpy="0 0 0"/>
+      <parent link="kitchen_counter_link" />
+      <child link="kitchen_counter_right_surface_link"/>
+    </joint>
+    <link name="kitchen_counter_right_surface_link">
+      <visual>
+        <geometry>
+          <box size="0.1 0.1 0.1"/>
+        </geometry>
+      </visual>
+    </link>
+    <joint name="${parent}_kitchen_counter_right_nav_goal_joint" type="fixed">
+      <origin xyz="0.6 0.55 0" rpy="0 0 0"/>
+      <parent link="kitchen_counter_link" />
+      <child link="kitchen_counter_right_nav_goal_link"/>
+    </joint>
+    <xacro:nav_goal prefix="kitchen_counter_right"/>
   </xacro:macro>
 </root>

File: urdf/kitchen_table.urdf.xacro (robot description, xacro)
@@ -3,5 +3,5 @@
   <xacro:macro name="kitchen_table" params="parent *origin">
     <joint name="${parent}_kitchen_table_joint" type="fixed">
-      <xacro:insert_block name="origin" />
+      <origin xyz="3.877 5.704 0" rpy="0 0 0" />
       <parent link="${parent}" />
       <child link="kitchen_table_link" />
@@ -9,5 +9,4 @@
     <link name="kitchen_table_link">
       <visual>
-        <origin xyz="1.111 0.228 0" rpy="0 0 0" />
         <geometry>
           <mesh filename="package://rail_collada_models/meshes/kitchen_table.dae" />
@@ -15,4 +14,23 @@
       </visual>
     </link>
+    <joint name="${parent}_kitchen_table_surface_joint" type="fixed">
+      <origin xyz="0 0 0.75" rpy="0 0 0"/>
+      <parent link="kitchen_table_link"/>
+      <child link="kitchen_table_surface_link"/>
+    </joint>
+      <link name="kitchen_table_surface_link">
+      <visual>
+        <geometry>
+          <box size="0.1 0.1 0.1"/>
+        </geometry>
+      </visual>
+    </link>
+    <!-- kitchen table nav goal, placed half of carl's length in front of the side near the couch-->
+    <joint name="${parent}_kitchen_table_nav_goal_1_joint" type="fixed">
+      <origin xyz="0 -.75 0" rpy="0 0 0"/>
+      <parent link="kitchen_table_link"/>
+      <child link="kitchen_table_nav_goal_link"/>
+    </joint>
+    <xacro:nav_goal prefix="kitchen_table"/>
   </xacro:macro>
 </root>

File: urdf/lab.urdf.xacro (robot description, xacro)
@@ -9,7 +9,7 @@
     <link name="lab_link">
       <visual>
-        <origin xyz="0 0 0" rpy="0 0 0" />
+        <origin xyz="-0.2 -0.15 0" rpy="0 0 0" />
         <geometry>
-<!--          <mesh filename="package://rail_collada_models/meshes/lab.dae" /> -->
+          <mesh filename="package://rail_collada_models/meshes/lab.dae" />
         </geometry>
       </visual>

File: urdf/lazy_chair_1.urdf.xacro (robot description, xacro)
@@ -1,7 +1,11 @@
+<!--
+NOT USED
+these should only be kept until russell and dave approve my macro use for the chairs
+-->
 <?xml version="1.0"?>
 <root xmlns:xacro="http://ros.org/wiki/xacro">
   <xacro:macro name="lazy_chair_1" params="parent *origin">
     <joint name="${parent}_lazy_chair_1_joint" type="fixed">
-      <xacro:insert_block name="origin" />
+      <origin xyz="3.64 1.1 0" rpy="0 0 0" />
       <parent link="${parent}" />
       <child link="lazy_chair_1_link" />
@@ -9,5 +13,4 @@
     <link name="lazy_chair_1_link">
       <visual>
-       <origin xyz="-.159 -4.349 0" rpy="0 0 0" />
         <geometry>
           <mesh filename="package://rail_collada_models/meshes/lazy_chair.dae" />
@@ -15,4 +18,10 @@
       </visual>
     </link>
+    <joint name="${parent}_lazy_chair_1_nav_goal" type="fixed">
+      <origin xyz="0 .84 0" rpy="0 0 0"/>
+      <parent link="lazy_chair_1_link"/>
+      <child link="lazy_chair_1_nav_goal_link"/>
+    </joint>
+    <xacro:nav_goal prefix="lazy_chair_1"/>
   </xacro:macro>
 </root>

File: urdf/lazy_chair_2.urdf.xacro (robot description, xacro)
@@ -1,7 +1,11 @@
+<!--
+NOT USED
+these should only be kept until russell and dave approve my macro use for the chairs
+-->
 <?xml version="1.0"?>
 <root xmlns:xacro="http://ros.org/wiki/xacro">
   <xacro:macro name="lazy_chair_2" params="parent *origin">
     <joint name="${parent}_lazy_chair_2_joint" type="fixed">
-      <xacro:insert_block name="origin" />
+      <origin xyz="2.62 1.1 0" rpy="0 0 0" />
       <parent link="${parent}" />
       <child link="lazy_chair_2_link" />
@@ -9,5 +13,4 @@
     <link name="lazy_chair_2_link">
       <visual>
-        <origin xyz="0.84 -4.341 0" rpy="0 0 0" />
         <geometry>
           <mesh filename="package://rail_collada_models/meshes/lazy_chair.dae" />
@@ -15,4 +18,10 @@
       </visual>
     </link>
+    <joint name="${parent}_lazy_chair_2_nav_goal" type="fixed">
+      <origin xyz="0 .84 0" rpy="0 0 0"/>
+      <parent link="lazy_chair_2_link"/>
+      <child link="lazy_chair_2_nav_goal_link"/>
+    </joint>
+    <xacro:nav_goal prefix="lazy_chair_1"/>
   </xacro:macro>
 </root>

File: urdf/left_shelves.urdf.xacro (robot description, xacro)
@@ -3,5 +3,5 @@
   <xacro:macro name="left_shelves" params="parent *origin">
     <joint name="${parent}_left_shelves_joint" type="fixed">
-      <xacro:insert_block name="origin" />
+      <origin xyz="0.425 0.838 0" rpy="0 0 ${-M_PI/2}" />
       <parent link="${parent}" />
       <child link="left_shelves_link" />
@@ -9,5 +9,4 @@
     <link name="left_shelves_link">
       <visual>
-        <origin xyz="-2.425 -4.712 0" rpy="0 0 ${-M_PI/2}" />
         <geometry>
           <mesh filename="package://rail_collada_models/meshes/left_shelves.dae" />
@@ -15,4 +14,22 @@
       </visual>
     </link>
+    <joint name="${parent}_left_shelves_low_joint" type="fixed">
+      <origin xyz="0 0 0.75" rpy="0 0 0"/>
+      <parent link="left_shelves_link"/>
+      <child link="left_shelves_low_shelf_link"/>
+    </joint>
+      <link name="left_shelves_low_shelf_link">
+      <visual>
+        <geometry>
+          <box size="0.1 0.1 0.1"/>
+        </geometry>
+      </visual>
+    </link>
+    <joint name="${parent}_left_shelves_nav_goal_joint" type="fixed">
+      <origin xyz="0 0.52 0" rpy="0 0 0"/>
+      <parent link="left_shelves_link"/>
+      <child link="left_shelves_nav_goal_link"/>
+    </joint>
+    <xacro:nav_goal prefix="left_shelves" />
   </xacro:macro>
 </root>

File: urdf/right_shelves.urdf.xacro (robot description, xacro)
@@ -3,5 +3,5 @@
   <xacro:macro name="right_shelves" params="parent *origin">
     <joint name="${parent}_right_shelves_joint" type="fixed">
-      <xacro:insert_block name="origin" />
+      <origin xyz="0.425 3.398 0" rpy="0 0 ${-M_PI/2}" />
       <parent link="${parent}" />
       <child link="right_shelves_link" />
@@ -9,5 +9,4 @@
     <link name="right_shelves_link">
       <visual>
-        <origin xyz="-2.435 -2.152 0" rpy="0 0 ${-M_PI/2}" />
         <geometry>
           <mesh filename="package://rail_collada_models/meshes/right_shelves.dae" />
@@ -15,4 +14,22 @@
       </visual>
     </link>
+    <joint name="${parent}_right_shelves_low_joint" type="fixed">
+      <origin xyz="0 0 0.51" rpy="0 0 0"/>
+      <parent link="right_shelves_link"/>
+      <child link="right_shelves_low_shelf_link"/>
+    </joint>
+      <link name="right_shelves_low_shelf_link">
+      <visual>
+        <geometry>
+          <box size="0.1 0.1 0.1"/>
+        </geometry>
+      </visual>
+    </link>
+   <joint name="${parent}_right_shelves_nav_goal_joint" type="fixed">
+      <origin xyz="0 0.52 0" rpy="0 0 0"/>
+      <parent link="right_shelves_link"/>
+      <child link="right_shelves_nav_goal_link"/>
+    </joint>
+    <xacro:nav_goal prefix="right_shelves"/>
   </xacro:macro>
 </root>

File: urdf/tv.urdf.xacro (robot description, xacro)
@@ -3,5 +3,5 @@
   <xacro:macro name="tv" params="parent *origin">
     <joint name="${parent}_tv_joint" type="fixed">
-      <xacro:insert_block name="origin" />
+      <origin xyz="0.89 2.1 0" rpy="0 0 ${-M_PI/2}" />
       <parent link="${parent}" />
       <child link="tv_link" />
@@ -9,5 +9,4 @@
     <link name="tv_link">
       <visual>
-        <origin xyz="-1.96 -3.45 0" rpy="0 0 ${-M_PI/2}" />
         <geometry>
           <mesh filename="package://rail_collada_models/meshes/tv.dae" />
@@ -15,4 +14,22 @@
       </visual>
     </link>
+    <joint name="${parent}_tv_surface_joint" type="fixed">
+      <origin xyz="0 0 0.605" rpy="0 0 0"/>
+      <parent link="tv_link"/>
+      <child link="tv_surface_link"/>
+    </joint>
+      <link name="tv_surface_link">
+      <visual>
+        <geometry>
+          <box size="0.1 0.1 0.1"/>
+        </geometry>
+      </visual>
+    </link>
+    <joint name="${parent}_tv_nav_goal_joint" type="fixed">
+      <origin xyz="0 0.7 0" rpy="0 0 0"/>
+      <parent link="tv_link"/>
+      <child link="tv_nav_goal_link"/>
+    </joint>
+    <xacro:nav_goal prefix="tv"/>
   </xacro:macro>
 </root>
