Commit message: turned nag goals to face objects. need to rotate all coordinate frames 180deg

File: urdf/coffee_table.urdf.xacro (robot description, xacro)
@@ -4,5 +4,5 @@
     <!-- Coffee table -->
     <joint name="${parent}_coffee_table_joint" type="fixed">
-      <origin xyz="3.345 2.99 0" rpy="0 0 ${M_PI/2}" />
+      <origin xyz="3.345 2.99 0" rpy="0 0 -${M_PI/2}" />
       <parent link="${parent}" />
       <child link="coffee_table_link" />
@@ -16,5 +16,5 @@
     </link>
     <joint name="${parent}_coffee_table_surface_joint" type="fixed">
-      <origin xyz="0 0 0.405" rpy="0 0 0"/>
+      <origin xyz="0 0 0.41" rpy="0 0 0"/>
       <parent link="coffee_table_link"/>
       <child link="coffee_table_surface_link"/>
@@ -29,5 +29,5 @@
     <!-- coffee table nav goal, placed half of carl's length in front of the long side near the coffee_table2-->
     <joint name="${parent}_coffee_table_nav_goal" type="fixed">
-      <origin xyz="0 0.6 0" rpy="0 0 0"/>
+      <origin xyz="0 -0.6 0" rpy="0 0 0"/>
       <parent link="coffee_table_link"/>
       <child link="coffee_table_nav_goal_link"/>

File: urdf/couch.urdf.xacro (robot description, xacro)
@@ -3,5 +3,5 @@
   <xacro:macro name="couch" params="parent *origin">
     <joint name="${parent}_couch_joint" type="fixed">
-      <xacro:insert_block name="origin" />
+      <origin xyz="4.497 2.94 0" rpy="0 0 ${M_PI/2}" />
       <parent link="${parent}" />
       <child link="couch_link" />
@@ -9,5 +9,4 @@
     <link name="couch_link">
       <visual>
-        <origin xyz="4.497 2.94 0" rpy="0 0 ${M_PI/2}" />
         <geometry>
           <mesh filename="package://rail_collada_models/meshes/couch.dae" />

File: urdf/kitchen_chair.urdf.xacro (robot description, xacro)
@@ -3,5 +3,5 @@
   <xacro:macro name="kitchen_chair" params="parent *origin">
     <joint name="${parent}_kitchen_chair_joint" type="fixed">
-      <xacro:insert_block name="origin" />
+      <origin xyz="3.345 5.775 0" rpy="0 0 ${-M_PI/2}" />
       <parent link="${parent}" />
       <child link="kitchen_chair_link" />
@@ -9,5 +9,4 @@
     <link name="kitchen_chair_link">
       <visual>
-        <origin xyz="3.345 5.775 0" rpy="0 0 ${-M_PI/2}" />
         <geometry>
           <mesh filename="package://rail_collada_models/meshes/kitchen_chair.dae" />

File: urdf/kitchen_counter.urdf.xacro (robot description, xacro)
@@ -22,13 +22,8 @@
     </joint>
     <link name="sink_link">
-      <visual>
-        <geometry>
-          <box size="0.1 0.1 0.1"/>
-        </geometry>
-      </visual>
     </link>
     <!-- Sink Nav Goal placed half of Carl's length in front of the middle of the sink-->
     <joint name="${parent}_sink_nav_goal_joint" type="fixed">
-      <origin xyz="0 0.55 0" rpy="0 0 0"/>
+      <origin xyz="0 0.55 0" rpy="0 0 ${M_PI}"/>
       <parent link="kitchen_counter_link" />
       <child link="sink_nav_goal_link"/>
@@ -42,12 +37,7 @@
     </joint>
     <link name="kitchen_counter_left_surface_link">
-      <visual>
-        <geometry>
-          <box size="0.1 0.1 0.1"/>
-        </geometry>
-      </visual>
     </link>
     <joint name= "${parent}_kitchen_counter_left_nav_goal_joint" type="fixed">
-      <origin xyz="-.6 0.55 0" rpy="0 0 0"/>
+      <origin xyz="-.6 0.55 0" rpy="0 0 ${M_PI}"/>
       <parent link="kitchen_counter_link" />
       <child link="kitchen_counter_left_nav_goal_link"/>
@@ -61,12 +51,7 @@
     </joint>
     <link name="kitchen_counter_right_surface_link">
-      <visual>
-        <geometry>
-          <box size="0.1 0.1 0.1"/>
-        </geometry>
-      </visual>
     </link>
     <joint name="${parent}_kitchen_counter_right_nav_goal_joint" type="fixed">
-      <origin xyz="0.6 0.55 0" rpy="0 0 0"/>
+      <origin xyz="0.6 0.55 0" rpy="0 0 ${M_PI}"/>
       <parent link="kitchen_counter_link" />
       <child link="kitchen_counter_right_nav_goal_link"/>

File: urdf/kitchen_table.urdf.xacro (robot description, xacro)
@@ -19,10 +19,5 @@
       <child link="kitchen_table_surface_link"/>
     </joint>
-      <link name="kitchen_table_surface_link">
-      <visual>
-        <geometry>
-          <box size="0.1 0.1 0.1"/>
-        </geometry>
-      </visual>
+    <link name="kitchen_table_surface_link">
     </link>
     <!-- kitchen table nav goal, placed half of carl's length in front of the side near the couch-->

File: urdf/lab.urdf.xacro (robot description, xacro)
@@ -3,5 +3,5 @@
   <xacro:macro name="lab" params="parent *origin">
     <joint name="${parent}_lab_joint" type="fixed">
-      <xacro:insert_block name="origin" />
+       <origin xyz="-0.2 -0.15 0" rpy="0 0 0" />
       <parent link="${parent}" />
       <child link="lab_link" />
@@ -9,5 +9,4 @@
     <link name="lab_link">
       <visual>
-        <origin xyz="-0.2 -0.15 0" rpy="0 0 0" />
         <geometry>
           <mesh filename="package://rail_collada_models/meshes/lab.dae" />

File: urdf/lazy_chairs.urdf.xacro (robot description, xacro)
@@ -22,10 +22,4 @@
       </visual>
     </link>
-    <joint name="${parent}_lazy_chair_${num}_nav_goal" type="fixed">
-      <origin xyz="0 .84 0" rpy="0 0 0"/>
-      <parent link="lazy_chair_${num}_link"/>
-      <child link="lazy_chair_${num}_nav_goal_link"/>
-    </joint>
-    <xacro:nav_goal prefix="lazy_chair_${num}"/>
   </xacro:macro>
 </root>

File: urdf/left_shelves.urdf.xacro (robot description, xacro)
@@ -14,18 +14,6 @@
       </visual>
     </link>
-    <joint name="${parent}_left_shelves_low_joint" type="fixed">
-      <origin xyz="0 0 0.75" rpy="0 0 0"/>
-      <parent link="left_shelves_link"/>
-      <child link="left_shelves_low_shelf_link"/>
-    </joint>
-      <link name="left_shelves_low_shelf_link">
-      <visual>
-        <geometry>
-          <box size="0.1 0.1 0.1"/>
-        </geometry>
-      </visual>
-    </link>
     <joint name="${parent}_left_shelves_nav_goal_joint" type="fixed">
-      <origin xyz="0 0.52 0" rpy="0 0 0"/>
+      <origin xyz="0 0.52 0" rpy="0 0 ${M_PI}"/>
       <parent link="left_shelves_link"/>
       <child link="left_shelves_nav_goal_link"/>

File: urdf/nav_goal.urdf.xacro (robot description, xacro)
@@ -3,9 +3,4 @@
   <xacro:macro name="nav_goal" params="prefix">
     <link name="${prefix}_nav_goal_link">
-      <visual>
-        <geometry>
-          <box size="0.1 0.1 0.01"/>
-        </geometry>
-      </visual>
     </link>
   </xacro:macro>

File: urdf/right_shelves.urdf.xacro (robot description, xacro)
@@ -14,18 +14,6 @@
       </visual>
     </link>
-    <joint name="${parent}_right_shelves_low_joint" type="fixed">
-      <origin xyz="0 0 0.51" rpy="0 0 0"/>
-      <parent link="right_shelves_link"/>
-      <child link="right_shelves_low_shelf_link"/>
-    </joint>
-      <link name="right_shelves_low_shelf_link">
-      <visual>
-        <geometry>
-          <box size="0.1 0.1 0.1"/>
-        </geometry>
-      </visual>
-    </link>
    <joint name="${parent}_right_shelves_nav_goal_joint" type="fixed">
-      <origin xyz="0 0.52 0" rpy="0 0 0"/>
+      <origin xyz="0 0.52 0" rpy="0 0 ${M_PI}"/>
       <parent link="right_shelves_link"/>
       <child link="right_shelves_nav_goal_link"/>

File: urdf/tv.urdf.xacro (robot description, xacro)
@@ -27,5 +27,5 @@
     </link>
     <joint name="${parent}_tv_nav_goal_joint" type="fixed">
-      <origin xyz="0 0.7 0" rpy="0 0 0"/>
+      <origin xyz="0 0.7 0" rpy="0 0 ${M_PI}"/>
       <parent link="tv_link"/>
       <child link="tv_nav_goal_link"/>

Commit message: added furniture and navgoal transforms

File: urdf/coffee_table.urdf.xacro (robot description, xacro)
@@ -20,10 +20,5 @@
       <child link="coffee_table_surface_link"/>
     </joint>
-      <link name="coffee_table_surface_link">
-      <visual>
-        <geometry>
-          <box size="0.1 0.1 0.1"/>
-        </geometry>
-      </visual>
+    <link name="coffee_table_surface_link">
     </link>
     <!-- coffee table nav goal, placed half of carl's length in front of the long side near the coffee_table2-->

File: urdf/tv.urdf.xacro (robot description, xacro)
@@ -19,10 +19,5 @@
       <child link="tv_surface_link"/>
     </joint>
-      <link name="tv_surface_link">
-      <visual>
-        <geometry>
-          <box size="0.1 0.1 0.1"/>
-        </geometry>
-      </visual>
+    <link name="tv_surface_link">
     </link>
     <joint name="${parent}_tv_nav_goal_joint" type="fixed">

Commit message: moved origins to ilab file and remove unnessecary lazy_chair code

File: urdf/coffee_table.urdf.xacro (robot description, xacro)
@@ -4,5 +4,5 @@
     <!-- Coffee table -->
     <joint name="${parent}_coffee_table_joint" type="fixed">
-      <origin xyz="3.345 2.99 0" rpy="0 0 -${M_PI/2}" />
+      <xacro:insert_block name="origin" />
       <parent link="${parent}" />
       <child link="coffee_table_link" />

File: urdf/couch.urdf.xacro (robot description, xacro)
@@ -3,5 +3,5 @@
   <xacro:macro name="couch" params="parent *origin">
     <joint name="${parent}_couch_joint" type="fixed">
-      <origin xyz="4.497 2.94 0" rpy="0 0 ${M_PI/2}" />
+      <xacro:insert_block name="origin" />
       <parent link="${parent}" />
       <child link="couch_link" />

File: urdf/ilab.urdf.xacro (robot description, xacro)
@@ -10,5 +10,5 @@
   <xacro:include filename="$(find rail_collada_models)/urdf/tv.urdf.xacro" />
   <xacro:include filename="$(find rail_collada_models)/urdf/left_shelves.urdf.xacro" />
-  <xacro:include filename="$(find rail_collada_models)/urdf/lazy_chairs.urdf.xacro" />
+  <xacro:include filename="$(find rail_collada_models)/urdf/lazy_chair.urdf.xacro" />
   <xacro:include filename="$(find rail_collada_models)/urdf/lab.urdf.xacro" />
   <xacro:property name="PARENT" value="map" />
@@ -24,32 +24,35 @@
   </joint>
   <xacro:lab parent="${FRAME}">
-    <origin xyz="0 0 0" rpy="0 0 0" />
+    <origin xyz="-0.2 -0.15 0" rpy="0 0 0" />
   </xacro:lab>
   <xacro:kitchen_counter parent="${FRAME}">
-    <origin xyz="0 0 0" rpy="0 0 0" />
+    <origin xyz="1.679 5.873 0" rpy="0 0 ${M_PI}"/>
   </xacro:kitchen_counter>
   <xacro:kitchen_table parent="${FRAME}">
-    <origin xyz="0 0 0" rpy="0 0 0" />
+    <origin xyz="3.877 5.704 0" rpy="0 0 0" />
   </xacro:kitchen_table>
   <xacro:coffee_table parent="${FRAME}">
-    <origin xyz="0 0 0" rpy="0 0 0" />
+    <origin xyz="3.345 2.99 0" rpy="0 0 -${M_PI/2}" />
   </xacro:coffee_table>
   <xacro:couch parent="${FRAME}">
-    <origin xyz="0 0 0" rpy="0 0 0" />
+    <origin xyz="4.497 2.94 0" rpy="0 0 ${M_PI/2}" />
   </xacro:couch>
   <xacro:right_shelves parent="${FRAME}">
-    <origin xyz="0 0 0" rpy="0 0 0" />
+    <origin xyz="0.425 3.398 0" rpy="0 0 ${-M_PI/2}" />
   </xacro:right_shelves>
   <xacro:tv parent="${FRAME}">
-    <origin xyz="0 0 0" rpy="0 0 0" />
+    <origin xyz="0.89 2.1 0" rpy="0 0 ${-M_PI/2}"/>
   </xacro:tv>
   <xacro:left_shelves parent="${FRAME}">
-    <origin xyz="0 0 0" rpy="0 0 0" />
+    <origin xyz="0.425 0.838 0" rpy="0 0 ${-M_PI/2}" />
   </xacro:left_shelves>
-  <xacro:lazy_chairs parent="${FRAME}">
-    <origin xyz="0 0 0" rpy="0 0 0" />
-  </xacro:lazy_chairs>
+  <xacro:lazy_chair parent="${FRAME}" suffix="1">
+    <origin xyz="3.64 1.1 0" rpy="0 0 0" />
+  </xacro:lazy_chair>
+  <xacro:lazy_chair parent="${FRAME}" suffix="2">
+    <origin xyz="2.621 1.1 0" rpy="0 0 0" />
+  </xacro:lazy_chair>
   <xacro:kitchen_chair parent="${FRAME}">
-    <origin xyz="0 0 0" rpy="0 0 0" />
+    <origin xyz="3.345 5.775 0" rpy="0 0 ${-M_PI/2}" />
   </xacro:kitchen_chair>
 </robot>

File: urdf/kitchen_chair.urdf.xacro (robot description, xacro)
@@ -3,5 +3,5 @@
   <xacro:macro name="kitchen_chair" params="parent *origin">
     <joint name="${parent}_kitchen_chair_joint" type="fixed">
-      <origin xyz="3.345 5.775 0" rpy="0 0 ${-M_PI/2}" />
+      <xacro:insert_block name="origin" />
       <parent link="${parent}" />
       <child link="kitchen_chair_link" />

File: urdf/kitchen_counter.urdf.xacro (robot description, xacro)
@@ -4,5 +4,5 @@
     <!--Kitchen Counter -->
     <joint name="${parent}_kitchen_counter_joint" type="fixed">
-      <origin xyz="1.679 5.873 0" rpy="0 0 ${M_PI}"/>
+      <xacro:insert_block name="origin" />
       <parent link="${parent}" />
       <child link="kitchen_counter_link"/>

File: urdf/kitchen_table.urdf.xacro (robot description, xacro)
@@ -3,5 +3,5 @@
   <xacro:macro name="kitchen_table" params="parent *origin">
     <joint name="${parent}_kitchen_table_joint" type="fixed">
-      <origin xyz="3.877 5.704 0" rpy="0 0 0" />
+      <xacro:insert_block name="origin" />
       <parent link="${parent}" />
       <child link="kitchen_table_link" />

File: urdf/lab.urdf.xacro (robot description, xacro)
@@ -3,5 +3,5 @@
   <xacro:macro name="lab" params="parent *origin">
     <joint name="${parent}_lab_joint" type="fixed">
-       <origin xyz="-0.2 -0.15 0" rpy="0 0 0" />
+      <xacro:insert_block name="origin" />
       <parent link="${parent}" />
       <child link="lab_link" />

File: urdf/left_shelves.urdf.xacro (robot description, xacro)
@@ -3,5 +3,5 @@
   <xacro:macro name="left_shelves" params="parent *origin">
     <joint name="${parent}_left_shelves_joint" type="fixed">
-      <origin xyz="0.425 0.838 0" rpy="0 0 ${-M_PI/2}" />
+      <xacro:insert_block name="origin" />
       <parent link="${parent}" />
       <child link="left_shelves_link" />

File: urdf/right_shelves.urdf.xacro (robot description, xacro)
@@ -3,5 +3,5 @@
   <xacro:macro name="right_shelves" params="parent *origin">
     <joint name="${parent}_right_shelves_joint" type="fixed">
-      <origin xyz="0.425 3.398 0" rpy="0 0 ${-M_PI/2}" />
+      <xacro:insert_block name="origin" />
       <parent link="${parent}" />
       <child link="right_shelves_link" />

File: urdf/tv.urdf.xacro (robot description, xacro)
@@ -3,5 +3,5 @@
   <xacro:macro name="tv" params="parent *origin">
     <joint name="${parent}_tv_joint" type="fixed">
-      <origin xyz="0.89 2.1 0" rpy="0 0 ${-M_PI/2}" />
+      <xacro:insert_block name="origin" />
       <parent link="${parent}" />
       <child link="tv_link" />

Commit message: remade nav goal macro

File: urdf/coffee_table.urdf.xacro (robot description, xacro)
@@ -22,11 +22,7 @@
     <link name="coffee_table_surface_link">
     </link>
-    <!-- coffee table nav goal, placed half of carl's length in front of the long side near the coffee_table2-->
-    <joint name="${parent}_coffee_table_nav_goal" type="fixed">
+    <xacro:nav_goal parent="coffee_table" child="coffee_table">
       <origin xyz="0 -0.6 0" rpy="0 0 0"/>
-      <parent link="coffee_table_link"/>
-      <child link="coffee_table_nav_goal_link"/>
-    </joint>
-    <xacro:nav_goal prefix="coffee_table"/>
+    </xacro:nav_goal>
   </xacro:macro>
 </root>

File: urdf/kitchen_counter.urdf.xacro (robot description, xacro)
@@ -21,13 +21,8 @@
       <child link="sink_link"/>
     </joint>
-    <link name="sink_link">
-    </link>
-    <!-- Sink Nav Goal placed half of Carl's length in front of the middle of the sink-->
-    <joint name="${parent}_sink_nav_goal_joint" type="fixed">
+    <link name="sink_link"/>
+    <xacro:nav_goal parent="sink" child="sink">
       <origin xyz="0 0.55 0" rpy="0 0 ${M_PI}"/>
-      <parent link="kitchen_counter_link" />
-      <child link="sink_nav_goal_link"/>
-    </joint>
-    <xacro:nav_goal prefix="sink"/>
+    </xacro:nav_goal>
     <!-- LEFT -->
     <joint name="${parent}_kitchen_counter_left_surface_joint" type="fixed">
@@ -38,10 +33,7 @@
     <link name="kitchen_counter_left_surface_link">
     </link>
-    <joint name= "${parent}_kitchen_counter_left_nav_goal_joint" type="fixed">
+    <xacro:nav_goal parent="kitchen_counter" child="kitchen_counter_left">
       <origin xyz="-.6 0.55 0" rpy="0 0 ${M_PI}"/>
-      <parent link="kitchen_counter_link" />
-      <child link="kitchen_counter_left_nav_goal_link"/>
-    </joint>
-    <xacro:nav_goal prefix="kitchen_counter_left"/>
+    </xacro:nav_goal>
     <!-- RIGHT -->
     <joint name="${parent}_kitchen_counter_right_surface_joint" type="fixed">
@@ -52,10 +44,7 @@
     <link name="kitchen_counter_right_surface_link">
     </link>
-    <joint name="${parent}_kitchen_counter_right_nav_goal_joint" type="fixed">
+    <xacro:nav_goal parent="kitchen_counter" child="kitchen_counter_right" >
       <origin xyz="0.6 0.55 0" rpy="0 0 ${M_PI}"/>
-      <parent link="kitchen_counter_link" />
-      <child link="kitchen_counter_right_nav_goal_link"/>
-    </joint>
-    <xacro:nav_goal prefix="kitchen_counter_right"/>
+    </xacro:nav_goal>
   </xacro:macro>
 </root>

File: urdf/kitchen_table.urdf.xacro (robot description, xacro)
@@ -21,11 +21,7 @@
     <link name="kitchen_table_surface_link">
     </link>
-    <!-- kitchen table nav goal, placed half of carl's length in front of the side near the couch-->
-    <joint name="${parent}_kitchen_table_nav_goal_1_joint" type="fixed">
+    <xacro:nav_goal parent="kitchen_table" child="kitchen_table">
       <origin xyz="0 -.75 0" rpy="0 0 0"/>
-      <parent link="kitchen_table_link"/>
-      <child link="kitchen_table_nav_goal_link"/>
-    </joint>
-    <xacro:nav_goal prefix="kitchen_table"/>
+    </xacro:nav_goal>
   </xacro:macro>
 </root>

File: urdf/left_shelves.urdf.xacro (robot description, xacro)
@@ -14,10 +14,7 @@
       </visual>
     </link>
-    <joint name="${parent}_left_shelves_nav_goal_joint" type="fixed">
+    <xacro:nav_goal parent="left_shelves" child="left_shelves">
       <origin xyz="0 0.52 0" rpy="0 0 ${M_PI}"/>
-      <parent link="left_shelves_link"/>
-      <child link="left_shelves_nav_goal_link"/>
-    </joint>
-    <xacro:nav_goal prefix="left_shelves" />
+    </xacro:nav_goal>
   </xacro:macro>
 </root>

File: urdf/nav_goal.urdf.xacro (robot description, xacro)
@@ -1,7 +1,11 @@
 <?xml version="1.0"?>
 <root xmlns:xacro="http://ros.org/wiki/xacro">
-  <xacro:macro name="nav_goal" params="prefix">
-    <link name="${prefix}_nav_goal_link">
-    </link>
+  <xacro:macro name="nav_goal" params="parent child *origin">
+  	<joint name="${child}_nav_goal_joint" type="fixed">
+      <xacro:insert_block name="origin" />
+      <parent link="${parent}_link"/>
+      <child link="${child}_nav_goal_link"/>
+    </joint>
+    <link name="${child}_nav_goal_link"/>
   </xacro:macro>
 </root>

File: urdf/right_shelves.urdf.xacro (robot description, xacro)
@@ -14,10 +14,7 @@
       </visual>
     </link>
-   <joint name="${parent}_right_shelves_nav_goal_joint" type="fixed">
+    <xacro:nav_goal parent="right_shelves" child="right_shelves">
       <origin xyz="0 0.52 0" rpy="0 0 ${M_PI}"/>
-      <parent link="right_shelves_link"/>
-      <child link="right_shelves_nav_goal_link"/>
-    </joint>
-    <xacro:nav_goal prefix="right_shelves"/>
+    </xacro:nav_goal>
   </xacro:macro>
 </root>

File: urdf/tv.urdf.xacro (robot description, xacro)
@@ -21,10 +21,7 @@
     <link name="tv_surface_link">
     </link>
-    <joint name="${parent}_tv_nav_goal_joint" type="fixed">
+    <xacro:nav_goal parent="tv" child="tv">
       <origin xyz="0 0.7 0" rpy="0 0 ${M_PI}"/>
-      <parent link="tv_link"/>
-      <child link="tv_nav_goal_link"/>
-    </joint>
-    <xacro:nav_goal prefix="tv"/>
+    </xacro:nav_goal>
   </xacro:macro>
 </root>

Commit message: using minified daes

File: urdf/coffee_table.urdf.xacro (robot description, xacro)
@@ -11,5 +11,5 @@
       <visual>
         <geometry>
-          <mesh filename="package://rail_collada_models/meshes/coffee_table.dae" />
+          <mesh filename="package://rail_collada_models/meshes/coffee_table.min.dae" />
         </geometry>
       </visual>

File: urdf/couch.urdf.xacro (robot description, xacro)
@@ -10,5 +10,5 @@
       <visual>
         <geometry>
-          <mesh filename="package://rail_collada_models/meshes/couch.dae" />
+          <mesh filename="package://rail_collada_models/meshes/couch.min.dae" />
         </geometry>
       </visual>

File: urdf/kitchen_chair.urdf.xacro (robot description, xacro)
@@ -10,5 +10,5 @@
       <visual>
         <geometry>
-          <mesh filename="package://rail_collada_models/meshes/kitchen_chair.dae" />
+          <mesh filename="package://rail_collada_models/meshes/kitchen_chair.min.dae" />
         </geometry>
       </visual>

File: urdf/kitchen_counter.urdf.xacro (robot description, xacro)
@@ -11,5 +11,5 @@
       <visual>
          <geometry>
-          <mesh filename="package://rail_collada_models/meshes/kitchen_counter.dae" />
+          <mesh filename="package://rail_collada_models/meshes/kitchen_counter.min.dae" />
         </geometry>
       </visual>

File: urdf/kitchen_table.urdf.xacro (robot description, xacro)
@@ -10,5 +10,5 @@
       <visual>
         <geometry>
-          <mesh filename="package://rail_collada_models/meshes/kitchen_table.dae" />
+          <mesh filename="package://rail_collada_models/meshes/kitchen_table.min.dae" />
         </geometry>
       </visual>

File: urdf/lab.urdf.xacro (robot description, xacro)
@@ -10,5 +10,5 @@
       <visual>
         <geometry>
-          <mesh filename="package://rail_collada_models/meshes/lab.dae" />
+          <mesh filename="package://rail_collada_models/meshes/lab.min.dae" />
         </geometry>
       </visual>

File: urdf/lazy_chair.urdf.xacro (robot description, xacro)
@@ -10,5 +10,5 @@
       <visual>
         <geometry>
-          <mesh filename="package://rail_collada_models/meshes/lazy_chair.dae" />
+          <mesh filename="package://rail_collada_models/meshes/lazy_chair.min.dae" />
         </geometry>
       </visual>

File: urdf/left_shelves.urdf.xacro (robot description, xacro)
@@ -10,5 +10,5 @@
       <visual>
         <geometry>
-          <mesh filename="package://rail_collada_models/meshes/left_shelves.dae" />
+          <mesh filename="package://rail_collada_models/meshes/left_shelves.min.dae" />
         </geometry>
       </visual>

File: urdf/right_shelves.urdf.xacro (robot description, xacro)
@@ -10,5 +10,5 @@
       <visual>
         <geometry>
-          <mesh filename="package://rail_collada_models/meshes/right_shelves.dae" />
+          <mesh filename="package://rail_collada_models/meshes/right_shelves.min.dae" />
         </geometry>
       </visual>

File: urdf/tv.urdf.xacro (robot description, xacro)
@@ -10,5 +10,5 @@
       <visual>
         <geometry>
-          <mesh filename="package://rail_collada_models/meshes/tv.dae" />
+          <mesh filename="package://rail_collada_models/meshes/tv.min.dae" />
         </geometry>
       </visual>

Commit message: added sizes of surfaces

File: urdf/coffee_table.urdf.xacro (robot description, xacro)
@@ -16,5 +16,6 @@
     </link>
     <xacro:surface parent="coffee_table" child="coffee_table">
-      <origin xyz="0 0 0.5" rpy="0 0 0"/>
+      <origin xyz="0 0 0.45" rpy="0 0 0"/>
+      <box size="1.2 0.5 0.05"/>
     </xacro:surface>
     <xacro:nav_goal parent="coffee_table" child="coffee_table">

File: urdf/kitchen_table.urdf.xacro (robot description, xacro)
@@ -16,4 +16,5 @@
     <xacro:surface parent="kitchen_table" child="kitchen_table">
       <origin xyz="0 0 0.75" rpy="0 0 0"/>
+      <box size="0.8 0.8 0.05"/>
     </xacro:surface>
     <xacro:nav_goal parent="kitchen_table" child="kitchen_table">
