Commit message: moved table marker closer

File: urdf/coffee_table.urdf.xacro (robot description, xacro)
@@ -20,5 +20,5 @@
     </xacro:surface>
     <xacro:nav_goal parent="coffee_table" child="coffee_table">
-      <origin xyz="0 -0.9 0" rpy="0 0 0"/>
+      <origin xyz="0 -0.8 0" rpy="0 0 0"/>
     </xacro:nav_goal>
   </xacro:macro>
