Commit message: added furniture models to room as robot model

File: urdf/ilab.urdf.xacro (robot description, xacro)
@@ -1,9 +1,18 @@
 <?xml version="1.0"?>
 <robot xmlns:xacro="http://www.ros.org/wiki/xacro" name="ilab">
-  <xacro:include filename="$(find rail_collada_models)/urdf/ikea_stool.urdf.xacro" />
-  <xacro:include filename="$(find rail_collada_models)/urdf/lab.urdf.xacro" />
+  <xacro:include filename="$(find rail_collada_models)/urdf/kitchen_counter.urdf.xacro" />
+  <xacro:include filename="$(find rail_collada_models)/urdf/kitchen_table.urdf.xacro" />
+  <xacro:include filename="$(find rail_collada_models)/urdf/coffee_table.urdf.xacro" />
+   <xacro:include filename="$(find rail_collada_models)/urdf/couch.urdf.xacro" />
+   <xacro:include filename="$(find rail_collada_models)/urdf/right_shelves.urdf.xacro" />
+   <xacro:include filename="$(find rail_collada_models)/urdf/tv.urdf.xacro" />
+   <xacro:include filename="$(find rail_collada_models)/urdf/left_shelves.urdf.xacro" />
+   <xacro:include filename="$(find rail_collada_models)/urdf/lazy_chair_1.urdf.xacro" />
+   <xacro:include filename="$(find rail_collada_models)/urdf/lazy_chair_2.urdf.xacro" />
+   <xacro:include filename="$(find rail_collada_models)/urdf/lab.urdf.xacro" />
   <xacro:property name="PARENT" value="map" />
   <xacro:property name="FRAME" value="ilab" />
-  <!-- fixed frame -->
+  <xacro:property name="M_PI" value="3.1415926535897931" />
+<!-- fixed frame -->
   <link name="${PARENT}" />
   <link name="${FRAME}" />
@@ -16,6 +25,30 @@
     <origin xyz="0 0 0" rpy="0 0 0" />
   </xacro:lab>
-  <xacro:ikea_stool parent="${FRAME}">
-    <origin xyz="0 0 0" rpy="0 0 0" />
-  </xacro:ikea_stool>
+  <xacro:kitchen_counter parent="${FRAME}">
+    <origin xyz="2.85 5.55 0" rpy="0 0 0" />
+  </xacro:kitchen_counter>
+  <xacro:kitchen_table parent="${FRAME}">
+    <origin xyz="2.85 5.55 0" rpy="0 0 0" />
+  </xacro:kitchen_table>
+  <xacro:coffee_table parent="${FRAME}">
+    <origin xyz="2.85 5.55 0" rpy="0 0 0" />
+  </xacro:coffee_table>
+  <xacro:couch parent="${FRAME}">
+    <origin xyz="2.85 5.55 0" rpy="0 0 0" />
+  </xacro:couch>
+  <xacro:right_shelves parent="${FRAME}">
+    <origin xyz="2.85 5.55 0" rpy="0 0 0" />
+  </xacro:right_shelves>
+  <xacro:tv parent="${FRAME}">
+    <origin xyz="2.85 5.55 0" rpy="0 0 0" />
+  </xacro:tv>
+  <xacro:left_shelves parent="${FRAME}">
+    <origin xyz="2.85 5.55 0" rpy="0 0 0" />
+  </xacro:left_shelves>
+  <xacro:lazy_chair_1 parent="${FRAME}">
+    <origin xyz="2.85 5.55 0" rpy="0 0 0" />
+  </xacro:lazy_chair_1>
+  <xacro:lazy_chair_2 parent="${FRAME}">
+    <origin xyz="2.85 5.55 0" rpy="0 0 0" />
+  </xacro:lazy_chair_2>
 </robot>

File: urdf/lab.urdf.xacro (robot description, xacro)
@@ -11,5 +11,5 @@
         <origin xyz="0 0 0" rpy="0 0 0" />
         <geometry>
-          <mesh filename="package://rail_collada_models/meshes/lab/lab.dae" />
+<!--          <mesh filename="package://rail_collada_models/meshes/lab.dae" /> -->
         </geometry>
       </visual>

Commit message: fixed lab position and floating marker

File: urdf/ilab.urdf.xacro (robot description, xacro)
@@ -24,5 +24,5 @@
   </joint>
   <xacro:lab parent="${FRAME}">
-    <origin xyz="-0.2 -0.15 0" rpy="0 0 0" />
+    <origin xyz="-0.15 0.0 0" rpy="0 0 0" />
   </xacro:lab>
   <xacro:kitchen_counter parent="${FRAME}">

File: urdf/kitchen_counter.urdf.xacro (robot description, xacro)
@@ -22,5 +22,5 @@
     </joint>
     <link name="sink_link"/>
-    <xacro:nav_goal parent="sink" child="sink">
+    <xacro:nav_goal parent="kitchen_counter" child="sink">
       <origin xyz="0 0.55 0" rpy="0 0 ${M_PI}"/>
     </xacro:nav_goal>

Commit message: fixed nav goals--chairs are flipped wrong direction

File: urdf/ilab.urdf.xacro (robot description, xacro)
@@ -27,5 +27,5 @@
   </xacro:lab>
   <xacro:kitchen_counter parent="${FRAME}">
-    <origin xyz="1.679 5.873 0" rpy="0 0 ${M_PI}"/>
+    <origin xyz="1.679 5.873 0" rpy="0 0 0"/>
   </xacro:kitchen_counter>
   <xacro:kitchen_table parent="${FRAME}">
@@ -36,15 +36,16 @@
   </xacro:coffee_table>
   <xacro:couch parent="${FRAME}">
-    <origin xyz="4.497 2.94 0" rpy="0 0 ${M_PI/2}" />
+    <origin xyz="4.497 2.94 0" rpy="0 0 ${-M_PI/2}" />
   </xacro:couch>
   <xacro:right_shelves parent="${FRAME}">
-    <origin xyz="0.425 3.398 0" rpy="0 0 ${-M_PI/2}" />
+    <origin xyz="0.425 3.398 0" rpy="0 0 ${M_PI/2}" />
   </xacro:right_shelves>
   <xacro:tv parent="${FRAME}">
-    <origin xyz="0.89 2.1 0" rpy="0 0 ${-M_PI/2}"/>
+    <origin xyz="0.89 2.1 0" rpy="0 0 ${M_PI/2}"/>
   </xacro:tv>
   <xacro:left_shelves parent="${FRAME}">
-    <origin xyz="0.425 0.838 0" rpy="0 0 ${-M_PI/2}" />
+    <origin xyz="0.425 0.838 0" rpy="0 0 ${M_PI/2}" />
   </xacro:left_shelves>
+<!-- THE CHAIRS FACE THE WRONG DIRECTION STILL-->
   <xacro:lazy_chair parent="${FRAME}" suffix="1">
     <origin xyz="3.64 1.1 0" rpy="0 0 0" />

File: urdf/kitchen_counter.urdf.xacro (robot description, xacro)
@@ -23,5 +23,5 @@
     <link name="sink_link"/>
     <xacro:nav_goal parent="kitchen_counter" child="sink">
-      <origin xyz="0 0.55 0" rpy="0 0 ${M_PI}"/>
+      <origin xyz="0 -0.55 0" rpy="0 0 0"/>
     </xacro:nav_goal>
     <!-- LEFT -->
@@ -34,5 +34,5 @@
     </link>
     <xacro:nav_goal parent="kitchen_counter" child="kitchen_counter_left">
-      <origin xyz="-.6 0.55 0" rpy="0 0 ${M_PI}"/>
+      <origin xyz="-.6 -0.55 0" rpy="0 0 0"/>
     </xacro:nav_goal>
     <!-- RIGHT -->
@@ -45,5 +45,5 @@
     </link>
     <xacro:nav_goal parent="kitchen_counter" child="kitchen_counter_right" >
-      <origin xyz="0.6 0.55 0" rpy="0 0 ${M_PI}"/>
+      <origin xyz="0.6 -0.55 0" rpy="0 0 0"/>
     </xacro:nav_goal>
   </xacro:macro>

File: urdf/left_shelves.urdf.xacro (robot description, xacro)
@@ -15,5 +15,5 @@
     </link>
     <xacro:nav_goal parent="left_shelves" child="left_shelves">
-      <origin xyz="0 0.52 0" rpy="0 0 ${M_PI}"/>
+      <origin xyz="0 -0.52 0" rpy="0 0 0"/>
     </xacro:nav_goal>
   </xacro:macro>

File: urdf/right_shelves.urdf.xacro (robot description, xacro)
@@ -15,5 +15,5 @@
     </link>
     <xacro:nav_goal parent="right_shelves" child="right_shelves">
-      <origin xyz="0 0.52 0" rpy="0 0 ${M_PI}"/>
+      <origin xyz="0 -0.52 0" rpy="0 0 0"/>
     </xacro:nav_goal>
   </xacro:macro>

File: urdf/tv.urdf.xacro (robot description, xacro)
@@ -22,5 +22,5 @@
     </link>
     <xacro:nav_goal parent="tv" child="tv">
-      <origin xyz="0 0.7 0" rpy="0 0 ${M_PI}"/>
+      <origin xyz="0 -0.7 0" rpy="0 0 0"/>
     </xacro:nav_goal>
   </xacro:macro>

Commit message: added surfaces with macro

File: urdf/ilab.urdf.xacro (robot description, xacro)
@@ -1,4 +1,6 @@
 <?xml version="1.0"?>
 <robot xmlns:xacro="http://www.ros.org/wiki/xacro" name="ilab">
+  <xacro:include filename="$(find rail_collada_models)/urdf/nav_goal.urdf.xacro" />
+  <xacro:include filename="$(find rail_collada_models)/urdf/surface.urdf.xacro" />
   <xacro:include filename="$(find rail_collada_models)/urdf/kitchen_counter.urdf.xacro" />
   <xacro:include filename="$(find rail_collada_models)/urdf/kitchen_chair.urdf.xacro" />
@@ -6,5 +8,4 @@
   <xacro:include filename="$(find rail_collada_models)/urdf/coffee_table.urdf.xacro" />
   <xacro:include filename="$(find rail_collada_models)/urdf/couch.urdf.xacro" />
-  <xacro:include filename="$(find rail_collada_models)/urdf/nav_goal.urdf.xacro" />
   <xacro:include filename="$(find rail_collada_models)/urdf/right_shelves.urdf.xacro" />
   <xacro:include filename="$(find rail_collada_models)/urdf/tv.urdf.xacro" />

File: urdf/kitchen_table.urdf.xacro (robot description, xacro)
@@ -14,11 +14,7 @@
       </visual>
     </link>
-    <joint name="${parent}_kitchen_table_surface_joint" type="fixed">
+    <xacro:surface parent="kitchen_table" child="kitchen_table">
       <origin xyz="0 0 0.75" rpy="0 0 0"/>
-      <parent link="kitchen_table_link"/>
-      <child link="kitchen_table_surface_link"/>
-    </joint>
-    <link name="kitchen_table_surface_link">
-    </link>
+    </xacro:surface>
     <xacro:nav_goal parent="kitchen_table" child="kitchen_table">
       <origin xyz="-1.00 0 0" rpy="0 0 -${M_PI/2}"/>

Commit message: flipped table surface. added chair surfaces

File: urdf/ilab.urdf.xacro (robot description, xacro)
@@ -48,5 +48,4 @@
     <origin xyz="0.425 0.838 0" rpy="0 0 ${M_PI/2}" />
   </xacro:left_shelves>
-<!-- THE CHAIRS FACE THE WRONG DIRECTION STILL-->
   <xacro:lazy_chair parent="${FRAME}" suffix="1">
     <origin xyz="3.64 1.1 0" rpy="0 0 ${M_PI}" />

File: urdf/kitchen_table.urdf.xacro (robot description, xacro)
@@ -15,5 +15,5 @@
     </link>
     <xacro:surface parent="kitchen_table" child="kitchen_table">
-      <origin xyz="0 0 0.75" rpy="0 0 0"/>
+      <origin xyz="0 0 0.75" rpy="0 0 -${M_PI/2}"/>
       <box size="0.8 0.8 0.05"/>
     </xacro:surface>
